Commit message: limit velocity

File: ros/kxr_models/urdf/kxr_test_head.urdf (robot description, URDF)
Before this commit: robot kxrl2l2a6h2m, 3 links, 2 joints
Joints:
- joint HEAD_JOINT1: limit lower=-2.0944 upper=2.0944 effort=0.656248 velocity=7.47998 -> lower=-2.0944 upper=2.0944 effort=0.656248 velocity=0.5
